Commit message: after dummy link fix

File: urdf/mybot.xacro (robot description, xacro)
@@ -2,6 +2,10 @@
 <robot name="mybot1" xmlns:xacro="http://www.ros.org/wiki/xacro">
 <xacro:include filename="$(find final_robot)/urdf/mybot.gazebo" />
-<!-- +++++++++++++++++++++++Robot Definition+++++++++++++++++++++++++ /-->
 <!--Chassis & Caster Link /-->
+<link name="base_footprint" />
+<joint name="base_footprint_joint" type="fixed">
+  <parent link="base_footprint" />
+  <child link="chassis" />
+</joint>
    <link name='chassis'>
    <visual name='chassis_visual'>
@@ -73,5 +77,4 @@
     <child link="weight_balance"/>
 </joint>
-<!-- ++++++++++++++++Left wheel+++++++++++++++++++++++++++++++ /-->
 <!--left wheel Link /-->
  <link name="left_wheel">
@@ -107,5 +110,4 @@
     <joint_properties damping="0.0" friction="0.0"/>
   </joint>
-<!-- +++++++++++++++++++ Right Wheel +++++++++++++++++++++++++++++++++ /-->
 <!--Right Wheel link /-->
   <link name="right_wheel">
@@ -141,5 +143,4 @@
     <joint_properties damping="0.0" friction="0.0"/>
   </joint>
-<!-- ++++++++++++++++++  Kinect  +++++++++++++++++++++++++++++ /-->
 <!--Kinect  Link /-->
 <link name="camera_link">
